File: Romi-unified-board-advanced.sch (KiCad schematic (older format))
At the start: 92 parts, among them J1 ServoAnalog, J10 LIDAR_DATA, J11 LIDAR_MOTOR, J12 ROMI-Encoder, J13 ROMI-Encoder, J14 THING, J15 THING, J16 SWD, J2 Conn_01x19_Female, J3 LineSensor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

Commit message: Finished schematic
Parts:
- J17: renamed from J?; footprint (none) -> Connector_JST:JST_PH_B2B-PH-K_1x02_P2.00mm_Vertical
- U10, U7: renamed from U?; footprint (none) -> US8:US8
- gave numbers to parts that had none: 11
Changed lines of the file:
@@
 GPIO25_B
 $Comp
-L power:+3.3V #PWR0102
+L power:+3.3V #PWR0112
 U 1 1 5F882560
 P 14150 16600
-F 0 "#PWR0102" H 14150 16450 50  0001 C CNN
+F 0 "#PWR0112" H 14150 16450 50  0001 C CNN
 F 1 "+3.3V" V 14165 16728 50  0000 L CNN
 F 2 "" H 14150 16600 50  0001 C CNN
@@
 GPIO25_B
 $Comp
-L Device:R_Small_US R?
+L Device:R_Small_US R11
 U 1 1 5FC4CE9A
 P 11100 20150
-F 0 "R?" H 11168 20196 50  0000 L CNN
+F 0 "R11" H 11168 20196 50  0000 L CNN
 F 1 "100k" H 11150 20050 50  0000 L CNN
 F 2 "Resistor_SMD:R_0603_1608Metric" H 11100 20150 50  0001 C CNN
@@
 $EndComp
 $Comp
-L Device:R_Small_US R?
+L Device:R_Small_US R12
 U 1 1 5FC4F62A
 P 11100 20500
-F 0 "R?" H 11168 20546 50  0000 L CNN
+F 0 "R12" H 11168 20546 50  0000 L CNN
 F 1 "100k" H 11150 20400 50  0000 L CNN
 F 2 "Resistor_SMD:R_0603_1608Metric" H 11100 20500 50  0001 C CNN
@@
 VSENSE_BAT
 $Comp
-L Regulator_Linear:SPX3819M5-L-3-3 U?
+L Regulator_Linear:SPX3819M5-L-3-3 U6
 U 1 1 5FCEC863
 P 15000 21700
-F 0 "U?" H 15000 22042 50  0000 C CNN
+F 0 "U6" H 15000 22042 50  0000 C CNN
 F 1 "SPX3819M5-L-3-3" H 15000 21951 50  0000 C CNN
 F 2 "Package_TO_SOT_SMD:SOT-23-5" H 15000 22025 50  0001 C CNN
@@
 $EndComp
 $Comp
-L power:+5V #PWR?
+L power:+5V #PWR0144
 U 1 1 5FCF1A67
 P 14250 21550
-F 0 "#PWR?" H 14250 21400 50  0001 C CNN
+F 0 "#PWR0144" H 14250 21400 50  0001 C CNN
 F 1 "+5V" H 14265 21723 50  0000 C CNN
 F 2 "" H 14250 21550 50  0001 C CNN
@@
 $EndComp
 $Comp
-L Device:R_Small_US R?
+L Device:R_Small_US R13
 U 1 1 5FCF2084
 P 14450 21700
-F 0 "R?" H 14518 21746 50  0000 L CNN
+F 0 "R13" H 14518 21746 50  0000 L CNN
 F 1 "100k" H 14500 21600 50  0000 L CNN
 F 2 "Resistor_SMD:R_0603_1608Metric" H 14450 21700 50  0001 C CNN
@@
 Connection ~ 14250 21600
 $Comp
-L power:GND #PWR?
+L power:GND #PWR0147
 U 1 1 5F81C713
 P 15000 22100
-F 0 "#PWR?" H 15000 21850 50  0001 C CNN
+F 0 "#PWR0147" H 15000 21850 50  0001 C CNN
 F 1 "GND" H 15005 21927 50  0000 C CNN
 F 2 "" H 15000 22100 50  0001 C CNN
@@
 $EndComp
 $Comp
-L power:+3.3V #PWR?
+L power:+3.3V #PWR0148
 U 1 1 5F81CD7C
 P 15650 21600
-F 0 "#PWR?" H 15650 21450 50  0001 C CNN
+F 0 "#PWR0148" H 15650 21450 50  0001 C CNN
 F 1 "+3.3V" V 15665 21728 50  0000 L CNN
 F 2 "" H 15650 21600 50  0001 C CNN
@@
 	15650 21600 15300 21600
 $Comp
-L Device:C C?
+L Device:C C16
 U 1 1 5F83FA41
 P 15500 21900
-F 0 "C?" H 15615 21946 50  0000 L CNN
+F 0 "C16" H 15615 21946 50  0000 L CNN
 F 1 "10nf" H 15615 21855 50  0000 L CNN
 F 2 "Capacitor_SMD:C_0603_1608Metric" H 15538 21750 50  0001 C CNN
@@
 $EndComp
 $Comp
-L power:GND #PWR?
+L power:GND #PWR0149
 U 1 1 5F840337
 P 15500 22100
-F 0 "#PWR?" H 15500 21850 50  0001 C CNN
+F 0 "#PWR0149" H 15500 21850 50  0001 C CNN
 F 1 "GND" H 15505 21927 50  0000 C CNN
 F 2 "" H 15500 22100 50  0001 C CNN
@@
 	15000 22000 15000 22100
 $Comp
-L Regulator_Linear:SPX3819M5-L U?
+L Regulator_Linear:SPX3819M5-L U11
 U 1 1 5F8A76E3
 P 16900 21700
-F 0 "U?" H 16900 22042 50  0000 C CNN
+F 0 "U11" H 16900 22042 50  0000 C CNN
 F 1 "SPX3819M5-L" H 16900 21951 50  0000 C CNN
 F 2 "Package_TO_SOT_SMD:SOT-23-5" H 16900 22025 50  0001 C CNN
@@
 $EndComp
 $Comp
-L power:+5V #PWR?
+L power:+5V #PWR0154
 U 1 1 5F8A920B
 P 16150 21550
-F 0 "#PWR?" H 16150 21400 50  0001 C CNN
+F 0 "#PWR0154" H 16150 21400 50  0001 C CNN
 F 1 "+5V" H 16165 21723 50  0000 C CNN
 F 2 "" H 16150 21550 50  0001 C CNN
@@
 $EndComp
 $Comp
-L Device:R_Small_US R?
+L Device:R_Small_US R26
 U 1 1 5F8A9211
 P 16350 21700
-F 0 "R?" H 16418 21746 50  0000 L CNN
+F 0 "R26" H 16418 21746 50  0000 L CNN
 F 1 "100k" H 16400 21600 50  0000 L CNN
 F 2 "Resistor_SMD:R_0603_1608Metric" H 16350 21700 50  0001 C CNN
@@
 Connection ~ 16150 21600
 $Comp
-L Device:R_Small_US R?
+L Device:R_Small_US R27
 U 1 1 5F8CB3FD
 P 17800 21750
-F 0 "R?" H 17868 21796 50  0000 L CNN
+F 0 "R27" H 17868 21796 50  0000 L CNN
 F 1 "100k" H 17850 21650 50  0000 L CNN
 F 2 "Resistor_SMD:R_0603_1608Metric" H 17800 21750 50  0001 C CNN
@@
 $EndComp
 $Comp
-L Device:R_Small_US R?
+L Device:R_Small_US R28
 U 1 1 5F8CC25F
 P 17800 22050
-F 0 "R?" H 17868 22096 50  0000 L CNN
+F 0 "R28" H 17868 22096 50  0000 L CNN
 F 1 "100k" H 17850 21950 50  0000 L CNN
 F 2 "Resistor_SMD:R_0603_1608Metric" H 17800 22050 50  0001 C CNN
@@
 $EndComp
 $Comp
-L power:GND #PWR?
+L power:GND #PWR0161
 U 1 1 5F8CC8A8
 P 16900 22050
-F 0 "#PWR?" H 16900 21800 50  0001 C CNN
+F 0 "#PWR0161" H 16900 21800 50  0001 C CNN
 F 1 "GND" H 16905 21877 50  0000 C CNN
 F 2 "" H 16900 22050 50  0001 C CNN
@@
 $EndComp
 $Comp
-L power:GND #PWR?
+L power:GND #PWR0162
 U 1 1 5F8CCC42
 P 17800 22200
-F 0 "#PWR?" H 17800 21950 50  0001 C CNN
+F 0 "#PWR0162" H 17800 21950 50  0001 C CNN
 F 1 "GND" H 17805 22027 50  0000 C CNN
 F 2 "" H 17800 22200 50  0001 C CNN
@@
 GPIO14_B
 $Comp
-L Device:C C?
+L Device:C C17
 U 1 1 5FAE64AE
 P 17450 22050
-F 0 "C?" H 17565 22096 50  0000 L CNN
+F 0 "C17" H 17565 22096 50  0000 L CNN
 F 1 "10nf" H 17565 22005 50  0000 L CNN
 F 2 "Capacitor_SMD:C_0603_1608Metric" H 17488 21900 50  0001 C CNN
@@
 Connection ~ 17450 21900
 $Comp
-L power:GND #PWR?
+L power:GND #PWR0163
 U 1 1 5FAE69D1
 P 17450 22200
-F 0 "#PWR?" H 17450 21950 50  0001 C CNN
+F 0 "#PWR0163" H 17450 21950 50  0001 C CNN
 F 1 "GND" H 17455 22027 50  0000 C CNN
 F 2 "" H 17450 22200 50  0001 C CNN
@@
 The Feather boards can't be\nsafley powered from a 5v source\nWe need a 4.2v "Fake Battery"
 $Comp
-L Connector:Conn_01x02_Female J?
+L Connector:Conn_01x02_Female J17
 U 1 1 5FAE93F9
 P 7450 21700
-F 0 "J?" H 7478 21676 50  0000 L CNN
+F 0 "J17" H 7478 21676 50  0000 L CNN
 F 1 "Conn_01x02_Female" H 7478 21585 50  0000 L CNN
-F 2 "" H 7450 21700 50  0001 C CNN
+F 2 "Connector_JST:JST_PH_B2B-PH-K_1x02_P2.00mm_Vertical" H 7450 21700 50  0001 C CNN
 F 3 "~" H 7450 21700 50  0001 C CNN
 	1    7450 21700
@@
 VFakeBAT
 $Comp
-L power:GND #PWR?
+L power:GND #PWR0171
 U 1 1 5FAEC927
 P 7150 21800
-F 0 "#PWR?" H 7150 21550 50  0001 C CNN
+F 0 "#PWR0171" H 7150 21550 50  0001 C CNN
 F 1 "GND" V 7155 21672 50  0000 R CNN
 F 2 "" H 7150 21800 50  0001 C CNN
@@
 GPIO36_B
 $Comp
-L TC7WB66CFK:TC7WB66CFK U?
+L TC7WB66CFK:TC7WB66CFK U10
 U 1 1 5FB62023
 P 15850 18050
-F 0 "U?" H 15825 18475 50  0000 C CNN
+F 0 "U10" H 15825 18475 50  0000 C CNN
 F 1 "TC7WB67CFK" H 15825 18384 50  0000 C CNN
-F 2 "" H 15850 17650 50  0001 C CNN
+F 2 "US8:US8" H 15850 17650 50  0001 C CNN
 F 3 "" H 15850 17650 50  0001 C CNN
 	1    15850 18050
@@
 LINE_CONN
 $Comp
-L 74xx:74AHC244 U?
+L 74xx:74AHC244 U5
 U 1 1 5FC71BD4
 P 11550 17450
-F 0 "U?" H 11300 18100 50  0000 C CNN
+F 0 "U5" H 11300 18100 50  0000 C CNN
 F 1 "74AHC244" H 11800 18100 50  0000 C CNN
 F 2 "Package_SO:TSSOP-20_4.4x6.5mm_P0.65mm" H 11550 17450 50  0001 C CNN
@@
 $EndComp
 $Comp
-L power:+3.3V #PWR?
+L power:+3.3V #PWR0178
 U 1 1 5FC9892F
 P 11550 16650
-F 0 "#PWR?" H 11550 16500 50  0001 C CNN
+F 0 "#PWR0178" H 11550 16500 50  0001 C CNN
 F 1 "+3.3V" V 11565 16778 50  0000 L CNN
 F 2 "" H 11550 16650 50  0001 C CNN
@@
 $EndComp
 $Comp
-L power:GND #PWR?
+L power:GND #PWR0179
 U 1 1 5FC98F23
 P 11550 18250
-F 0 "#PWR?" H 11550 18000 50  0001 C CNN
+F 0 "#PWR0179" H 11550 18000 50  0001 C CNN
 F 1 "GND" V 11555 18122 50  0000 R CNN
 F 2 "" H 11550 18250 50  0001 C CNN
@@
 GPIO17
 $Comp
-L TC7WB66CFK:TC7WB66CFK U?
+L TC7WB66CFK:TC7WB66CFK U7
 U 1 1 5FCE9A3D
 P 15850 17050
-F 0 "U?" H 15825 17475 50  0000 C CNN
+F 0 "U7" H 15825 17475 50  0000 C CNN
 F 1 "TC7WB67CFK" H 15825 17384 50  0000 C CNN
-F 2 "" H 15850 16650 50  0001 C CNN
+F 2 "US8:US8" H 15850 16650 50  0001 C CNN
 F 3 "" H 15850 16650 50  0001 C CNN
 	1    15850 17050
